File: KiCad/cassin_pwr2.kicad_pcb (KiCad board)
At the start: 2 copper layers, 68.6 x 53.3 mm, 31 parts, among them J1 Conn_01x03_Male, J2 Screw_Terminal_01x02, J3 Screw_Terminal_01x02, J4 Conn_01x03_Male, J5 Conn_01x04_Male, P1 Power, P2 Analog, P3 Digital, P4 Digital, P5 CONN_01X01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

Commit message: fabversion
Parts:
- removed P5, P6, P7, P8: CONN_01X01, Socket_Arduino_Uno:Arduino_1pin
- added kibuzzard-628A722A: G***, kibuzzard-628A722A, B.Cu at (150.1, 80.1)
- moved R4 1.27 mm to (166.9, 106.0)
- moved R5 1.27 mm to (170.7, 116.2)
Routing:
- net GND: track 38.0 -> 18.2 mm
- net /A3: track 25.8 -> 31.2 mm
- net /Vin: track 47.8 -> 52.4 mm
- net /A2: track 24.0 -> 26.0 mm
- net /A0: track 12.3 -> 13.5 mm
- net /Vmot: track 86.1 -> 87.0 mm
